Commit message: Update open_manipulator_x_arm.urdf.xacro
카메라 위치 변경

Signed-off-by: DSCL-CHO <wptjcks15@gmail.com>

File: open_manipulator_description/urdf/om_x/open_manipulator_x_arm.urdf.xacro (robot description, xacro)
@@ -240,5 +240,5 @@
     <!-- Gripper camera -->
     <joint type="fixed" name="${prefix}gripper_camera_joint">
-      <origin xyz="0.08 0.0 0.0" rpy="0 0 0"/>
+      <origin xyz="0.08 0.0 0.05" rpy="0 0 0"/>
       <child link="${prefix}gripper_camera_link"/>
       <parent link="${prefix}link5"/>
